File: lucud/pcb/Power.sch (KiCad schematic (older format))
At the start: 5 parts, among them J1 Conn_02x05_Odd_Even, U2 R-78E3.3-0.5

Commit message: Moved some shit around, changed the spec, worked on the PCB
Parts:
- C1, C3: value 1uF -> 1uF 25V
- C2: value 1uF -> 1uF 6.3V
Changed lines of the file:
@@
 $Descr A4 11693 8268
 encoding utf-8
-Sheet 3 3
+Sheet 3 4
 Title ""
 Date ""
@@
 P 6850 4050
 F 0 "C2" H 7028 4096 50  0000 L CNN
-F 1 "1uF" H 7028 4005 50  0000 L CNN
+F 1 "1uF 6.3V" H 7028 4005 50  0000 L CNN
 F 2 "Capacitor_SMD:C_0603_1608Metric" H 6850 4050 50  0001 C CNN
 F 3 "~" H 6850 4050 50  0001 C CNN
@@
 P 4750 4050
 F 0 "C1" H 4928 4096 50  0000 L CNN
-F 1 "1uF" H 4928 4005 50  0000 L CNN
+F 1 "1uF 25V" H 4928 4005 50  0000 L CNN
 F 2 "Capacitor_SMD:C_0603_1608Metric" H 4750 4050 50  0001 C CNN
 F 3 "~" H 4750 4050 50  0001 C CNN
@@
 P 3100 3450
 F 0 "C3" H 3278 3496 50  0000 L CNN
-F 1 "1uF" H 3278 3405 50  0000 L CNN
+F 1 "1uF 25V" H 3278 3405 50  0000 L CNN
 F 2 "Capacitor_SMD:C_0603_1608Metric" H 3100 3450 50  0001 C CNN
 F 3 "~" H 3100 3450 50  0001 C CNN

Commit message: Worked on the PCB
Parts:
- added C10: 1uF 25V, Capacitor_SMD:C_0603_1608Metric, symbol pspice:CAP
- added C11: 1uF 6.3V, Capacitor_SMD:C_0603_1608Metric, symbol pspice:CAP
- added U5: R-78E5.0-0.5, Converter_DCDC:Converter_DCDC_RECOM_R-78E-0.5_THT, symbol Regulator_Switching:R-78E5.0-0.5
Connections:
- net +12V: now also C10.1, U5.1 (IN)
- net GND: now also C10.2, C11.2, U5.2 (GND)
- new net +5V: C11.1, U5.3 (OUT)
Other:
- moved on the sheet: C1, C2, U2
Changed lines of the file:
@@
 $Descr A4 11693 8268
 encoding utf-8
-Sheet 3 4
+Sheet 3 5
 Title ""
 Date ""
@@
 L Regulator_Switching:R-78E3.3-0.5 U2
 U 1 1 5C243CB2
-P 5850 3600
-F 0 "U2" H 5850 3842 50  0000 C CNN
-F 1 "R-78E3.3-0.5" H 5850 3751 50  0000 C CNN
-F 2 "Converter_DCDC:Converter_DCDC_RECOM_R-78E-0.5_THT" H 5900 3350 50  0001 L CIN
-F 3 "https://www.recom-power.com/pdf/Innoline/R-78Exx-0.5.pdf" H 5850 3600 50  0001 C CNN
-	1    5850 3600
+P 5850 4800
+F 0 "U2" H 5850 5042 50  0000 C CNN
+F 1 "R-78E3.3-0.5" H 5850 4951 50  0000 C CNN
+F 2 "Converter_DCDC:Converter_DCDC_RECOM_R-78E-0.5_THT" H 5900 4550 50  0001 L CIN
+F 3 "https://www.recom-power.com/pdf/Innoline/R-78Exx-0.5.pdf" H 5850 4800 50  0001 C CNN
+	1    5850 4800
 	1    0    0    -1
 $EndComp
@@
 L pspice:CAP C2
 U 1 1 5C2441A0
-P 6850 4050
-F 0 "C2" H 7028 4096 50  0000 L CNN
-F 1 "1uF 6.3V" H 7028 4005 50  0000 L CNN
-F 2 "Capacitor_SMD:C_0603_1608Metric" H 6850 4050 50  0001 C CNN
-F 3 "~" H 6850 4050 50  0001 C CNN
-	1    6850 4050
+P 6850 5250
+F 0 "C2" H 7028 5296 50  0000 L CNN
+F 1 "1uF 6.3V" H 7028 5205 50  0000 L CNN
+F 2 "Capacitor_SMD:C_0603_1608Metric" H 6850 5250 50  0001 C CNN
+F 3 "~" H 6850 5250 50  0001 C CNN
+	1    6850 5250
 	1    0    0    -1
 $EndComp
@@
 L pspice:CAP C1
 U 1 1 5C2441F8
-P 4750 4050
-F 0 "C1" H 4928 4096 50  0000 L CNN
-F 1 "1uF 25V" H 4928 4005 50  0000 L CNN
-F 2 "Capacitor_SMD:C_0603_1608Metric" H 4750 4050 50  0001 C CNN
-F 3 "~" H 4750 4050 50  0001 C CNN
-	1    4750 4050
-	1    0    0    -1
-$EndComp
-Wire Wire Line
-	5550 3600 4750 3600
-Wire Wire Line
-	4750 3800 4750 3600
-Connection ~ 4750 3600
-Wire Wire Line
-	4750 3600 4550 3600
-Wire Wire Line
-	6150 3600 6850 3600
-Wire Wire Line
-	6850 3800 6850 3600
-Connection ~ 6850 3600
-Wire Wire Line
-	6850 3600 7050 3600
-Wire Wire Line
-	5850 3900 5850 4500
-Wire Wire Line
-	4750 4300 4750 4500
-Wire Wire Line
-	4750 4500 5850 4500
-Connection ~ 5850 4500
-Wire Wire Line
-	6850 4300 6850 4500
-Wire Wire Line
-	6850 4500 5850 4500
+P 4750 5250
+F 0 "C1" H 4928 5296 50  0000 L CNN
+F 1 "1uF 25V" H 4928 5205 50  0000 L CNN
+F 2 "Capacitor_SMD:C_0603_1608Metric" H 4750 5250 50  0001 C CNN
+F 3 "~" H 4750 5250 50  0001 C CNN
+	1    4750 5250
+	1    0    0    -1
+$EndComp
+Wire Wire Line
+	5550 4800 4750 4800
+Wire Wire Line
+	4750 5000 4750 4800
+Connection ~ 4750 4800
+Wire Wire Line
+	4750 4800 4550 4800
+Wire Wire Line
+	6150 4800 6850 4800
+Wire Wire Line
+	6850 5000 6850 4800
+Connection ~ 6850 4800
+Wire Wire Line
+	6850 4800 7050 4800
+Wire Wire Line
+	5850 5100 5850 5700
+Wire Wire Line
+	4750 5500 4750 5700
+Wire Wire Line
+	4750 5700 5850 5700
+Connection ~ 5850 5700
+Wire Wire Line
+	6850 5500 6850 5700
+Wire Wire Line
+	6850 5700 5850 5700
 $Comp
 L power:GND #PWR01
 U 1 1 5C2443CA
-P 5850 4750
-F 0 "#PWR01" H 5850 4500 50  0001 C CNN
-F 1 "GND" H 5855 4577 50  0000 C CNN
-F 2 "" H 5850 4750 50  0001 C CNN
-F 3 "" H 5850 4750 50  0001 C CNN
-	1    5850 4750
-	1    0    0    -1
-$EndComp
-Wire Wire Line
-	5850 4500 5850 4750
+P 5850 5950
+F 0 "#PWR01" H 5850 5700 50  0001 C CNN
+F 1 "GND" H 5855 5777 50  0000 C CNN
+F 2 "" H 5850 5950 50  0001 C CNN
+F 3 "" H 5850 5950 50  0001 C CNN
+	1    5850 5950
+	1    0    0    -1
+$EndComp
+Wire Wire Line
+	5850 5700 5850 5950
 $Comp
 L power:+12V #PWR07
 U 1 1 5C244519
-P 4550 3450
-F 0 "#PWR07" H 4550 3300 50  0001 C CNN
-F 1 "+12V" H 4565 3623 50  0000 C CNN
-F 2 "" H 4550 3450 50  0001 C CNN
-F 3 "" H 4550 3450 50  0001 C CNN
-	1    4550 3450
-	1    0    0    -1
-$EndComp
-Wire Wire Line
-	4550 3450 4550 3600
+P 4550 4650
+F 0 "#PWR07" H 4550 4500 50  0001 C CNN
+F 1 "+12V" H 4565 4823 50  0000 C CNN
+F 2 "" H 4550 4650 50  0001 C CNN
+F 3 "" H 4550 4650 50  0001 C CNN
+	1    4550 4650
+	1    0    0    -1
+$EndComp
+Wire Wire Line
+	4550 4650 4550 4800
 $Comp
 L power:+3.3V #PWR08
 U 1 1 5C2448FE
-P 7050 3450
-F 0 "#PWR08" H 7050 3300 50  0001 C CNN
-F 1 "+3.3V" H 7065 3623 50  0000 C CNN
-F 2 "" H 7050 3450 50  0001 C CNN
-F 3 "" H 7050 3450 50  0001 C CNN
-	1    7050 3450
-	1    0    0    -1
-$EndComp
-Wire Wire Line
-	7050 3450 7050 3600
+P 7050 4650
+F 0 "#PWR08" H 7050 4500 50  0001 C CNN
+F 1 "+3.3V" H 7065 4823 50  0000 C CNN
+F 2 "" H 7050 4650 50  0001 C CNN
+F 3 "" H 7050 4650 50  0001 C CNN
+	1    7050 4650
+	1    0    0    -1
+$EndComp
+Wire Wire Line
+	7050 4650 7050 4800
 $Comp
 L Connector_Generic:Conn_02x05_Odd_Even J1
@@
 Wire Wire Line
 	3100 3200 3100 3150
+$Comp
+L Regulator_Switching:R-78E5.0-0.5 U5
+U 1 1 5C2D5DAF
+P 5850 2750
+F 0 "U5" H 5850 2992 50  0000 C CNN
+F 1 "R-78E5.0-0.5" H 5850 2901 50  0000 C CNN
+F 2 "Converter_DCDC:Converter_DCDC_RECOM_R-78E-0.5_THT" H 5900 2500 50  0001 L CIN
+F 3 "https://www.recom-power.com/pdf/Innoline/R-78Exx-0.5.pdf" H 5850 2750 50  0001 C CNN
+	1    5850 2750
+	1    0    0    -1
+$EndComp
+$Comp
+L pspice:CAP C11
+U 1 1 5C2D63BD
+P 6850 3200
+F 0 "C11" H 7028 3246 50  0000 L CNN
+F 1 "1uF 6.3V" H 7028 3155 50  0000 L CNN
+F 2 "Capacitor_SMD:C_0603_1608Metric" H 6850 3200 50  0001 C CNN
+F 3 "~" H 6850 3200 50  0001 C CNN
+	1    6850 3200
+	1    0    0    -1
+$EndComp
+$Comp
+L pspice:CAP C10
+U 1 1 5C2D63C4
+P 4750 3200
+F 0 "C10" H 4928 3246 50  0000 L CNN
+F 1 "1uF 25V" H 4928 3155 50  0000 L CNN
+F 2 "Capacitor_SMD:C_0603_1608Metric" H 4750 3200 50  0001 C CNN
+F 3 "~" H 4750 3200 50  0001 C CNN
+	1    4750 3200
+	1    0    0    -1
+$EndComp
+Wire Wire Line
+	5550 2750 4750 2750
+Wire Wire Line
+	4750 2950 4750 2750
+Connection ~ 4750 2750
+Wire Wire Line
+	4750 2750 4550 2750
+Wire Wire Line
+	6150 2750 6850 2750
+Wire Wire Line
+	6850 2950 6850 2750
+Connection ~ 6850 2750
+Wire Wire Line
+	6850 2750 7050 2750
+Wire Wire Line
+	5850 3050 5850 3650
+Wire Wire Line
+	4750 3450 4750 3650
+Wire Wire Line
+	4750 3650 5850 3650
+Connection ~ 5850 3650
+Wire Wire Line
+	6850 3450 6850 3650
+Wire Wire Line
+	6850 3650 5850 3650
+$Comp
+L power:GND #PWR027
+U 1 1 5C2D63D9
+P 5850 3900
+F 0 "#PWR027" H 5850 3650 50  0001 C CNN
+F 1 "GND" H 5855 3727 50  0000 C CNN
+F 2 "" H 5850 3900 50  0001 C CNN
+F 3 "" H 5850 3900 50  0001 C CNN
+	1    5850 3900
+	1    0    0    -1
+$EndComp
+Wire Wire Line
+	5850 3650 5850 3900
+$Comp
+L power:+12V #PWR026
+U 1 1 5C2D63E0
+P 4550 2600
+F 0 "#PWR026" H 4550 2450 50  0001 C CNN
+F 1 "+12V" H 4565 2773 50  0000 C CNN
+F 2 "" H 4550 2600 50  0001 C CNN
+F 3 "" H 4550 2600 50  0001 C CNN
+	1    4550 2600
+	1    0    0    -1
+$EndComp
+Wire Wire Line
+	4550 2600 4550 2750
+Wire Wire Line
+	7050 2600 7050 2750
+$Comp
+L power:+5V #PWR028
+U 1 1 5C2D6BBC
+P 7050 2600
+F 0 "#PWR028" H 7050 2450 50  0001 C CNN
+F 1 "+5V" H 7065 2773 50  0000 C CNN
+F 2 "" H 7050 2600 50  0001 C CNN
+F 3 "" H 7050 2600 50  0001 C CNN
+	1    7050 2600
+	1    0    0    -1
+$EndComp
 $EndSCHEMATC
