File: lucud/pcb/DO-Buffer.sch (KiCad schematic (older format))
At the start: 4 parts, among them U3 74LVC125, U4 74LVC125

Commit message: Added buffer parts
Parts:
- U3: footprint (none) -> Package_SO:SOIC-14_3.9x8.7mm_P1.27mm; Part Number (none) -> 74LVC125AD,118
- U3, U4: footprint (none) -> Package_SO:SOIC-14_3.9x8.7mm_P1.27mm
Changed lines of the file:
@@
 F 0 "U3" H 4950 3167 50  0000 C CNN
 F 1 "74LVC125" H 4950 3076 50  0000 C CNN
-F 2 "" H 4950 2850 50  0001 C CNN
+F 2 "Package_SO:SOIC-14_3.9x8.7mm_P1.27mm" H 4950 2850 50  0001 C CNN
 F 3 "http://www.ti.com/lit/gpn/sn74LVC125" H 4950 2850 50  0001 C CNN
+F 4 "74LVC125AD,118" H 4950 2850 50  0001 C CNN "Part Number"
 	1    4950 2850
 	-1   0    0    -1
@@
 F 0 "U3" H 4950 3917 50  0000 C CNN
 F 1 "74LVC125" H 4950 3826 50  0000 C CNN
-F 2 "" H 4950 3600 50  0001 C CNN
+F 2 "Package_SO:SOIC-14_3.9x8.7mm_P1.27mm" H 4950 3600 50  0001 C CNN
 F 3 "http://www.ti.com/lit/gpn/sn74LVC125" H 4950 3600 50  0001 C CNN
 	2    4950 3600
@@
 F 0 "U3" H 4950 4667 50  0000 C CNN
 F 1 "74LVC125" H 4950 4576 50  0000 C CNN
-F 2 "" H 4950 4350 50  0001 C CNN
+F 2 "Package_SO:SOIC-14_3.9x8.7mm_P1.27mm" H 4950 4350 50  0001 C CNN
 F 3 "http://www.ti.com/lit/gpn/sn74LVC125" H 4950 4350 50  0001 C CNN
 	3    4950 4350
@@
 F 0 "U3" H 4950 5417 50  0000 C CNN
 F 1 "74LVC125" H 4950 5326 50  0000 C CNN
-F 2 "" H 4950 5100 50  0001 C CNN
+F 2 "Package_SO:SOIC-14_3.9x8.7mm_P1.27mm" H 4950 5100 50  0001 C CNN
 F 3 "http://www.ti.com/lit/gpn/sn74LVC125" H 4950 5100 50  0001 C CNN
 	4    4950 5100
@@
 F 0 "U3" H 1630 1696 50  0000 L CNN
 F 1 "74LVC125" H 1630 1605 50  0000 L CNN
-F 2 "" H 1400 1650 50  0001 C CNN
+F 2 "Package_SO:SOIC-14_3.9x8.7mm_P1.27mm" H 1400 1650 50  0001 C CNN
 F 3 "http://www.ti.com/lit/gpn/sn74LVC125" H 1400 1650 50  0001 C CNN
 	5    1400 1650
@@
 F 0 "U4" H 7400 3117 50  0000 C CNN
 F 1 "74LVC125" H 7400 3026 50  0000 C CNN
-F 2 "" H 7400 2800 50  0001 C CNN
+F 2 "Package_SO:SOIC-14_3.9x8.7mm_P1.27mm" H 7400 2800 50  0001 C CNN
 F 3 "http://www.ti.com/lit/gpn/sn74LVC125" H 7400 2800 50  0001 C CNN
 	1    7400 2800
@@
 F 0 "U4" H 7400 3867 50  0000 C CNN
 F 1 "74LVC125" H 7400 3776 50  0000 C CNN
-F 2 "" H 7400 3550 50  0001 C CNN
+F 2 "Package_SO:SOIC-14_3.9x8.7mm_P1.27mm" H 7400 3550 50  0001 C CNN
 F 3 "http://www.ti.com/lit/gpn/sn74LVC125" H 7400 3550 50  0001 C CNN
 	2    7400 3550
@@
 F 0 "U4" H 7400 4617 50  0000 C CNN
 F 1 "74LVC125" H 7400 4526 50  0000 C CNN
-F 2 "" H 7400 4300 50  0001 C CNN
+F 2 "Package_SO:SOIC-14_3.9x8.7mm_P1.27mm" H 7400 4300 50  0001 C CNN
 F 3 "http://www.ti.com/lit/gpn/sn74LVC125" H 7400 4300 50  0001 C CNN
 	3    7400 4300
@@
 F 0 "U4" H 7400 5367 50  0000 C CNN
 F 1 "74LVC125" H 7400 5276 50  0000 C CNN
-F 2 "" H 7400 5050 50  0001 C CNN
+F 2 "Package_SO:SOIC-14_3.9x8.7mm_P1.27mm" H 7400 5050 50  0001 C CNN
 F 3 "http://www.ti.com/lit/gpn/sn74LVC125" H 7400 5050 50  0001 C CNN
 	4    7400 5050
@@
 F 0 "U4" H 3130 1696 50  0000 L CNN
 F 1 "74LVC125" H 3130 1605 50  0000 L CNN
-F 2 "" H 2900 1650 50  0001 C CNN
+F 2 "Package_SO:SOIC-14_3.9x8.7mm_P1.27mm" H 2900 1650 50  0001 C CNN
 F 3 "http://www.ti.com/lit/gpn/sn74LVC125" H 2900 1650 50  0001 C CNN
 	5    2900 1650
